Commit message: support toroboeye-0.9.0 at noetic-devel

File: toroboeye_description/urdf/sl80.urdf.xacro (robot description, xacro)
@@ -12,27 +12,9 @@
     <visual>
       <geometry>
-        <mesh filename="package://toroboeye_description/meshes/SL40.stl" scale="0.001 0.001 0.001"/>
+        <mesh filename="package://toroboeye_description/meshes/SL80.stl" scale="0.001 0.001 0.001"/>
       </geometry>
-      <origin xyz="0 0 0" rpy="0 0 ${90*M_PI/180}"/>
+      <origin xyz="-0.037 0.04 -0.021056" rpy="0 0 ${90*M_PI/180}"/>
       <material name="gray">
         <color rgba="0.8 0.8 0.8 1.0"/>
-      </material>
-    </visual>
-    <visual>
-      <geometry>
-        <cylinder radius="0.012" length="0.003"/>
-      </geometry>
-      <origin xyz="0 0 0.016" rpy="0 ${90*M_PI/180} 0"/>
-      <material name="black">
-        <color rgba="0.6 0.6 0.6 1.0"/>
-      </material>
-    </visual>
-    <visual>
-      <geometry>
-        <cylinder radius="0.01" length="0.003"/>
-      </geometry>
-      <origin xyz="0 0 0.056" rpy="0 ${90*M_PI/180} 0"/>
-      <material name="black">
-        <color rgba="0.6 0.6 0.6 1.0"/>
       </material>
     </visual>
@@ -48,5 +30,5 @@
     <parent link="$(arg prefix)/camera_frame"/>
     <child  link="$(arg prefix)/camera_optical_frame"/>
-    <origin xyz="0 0 0" rpy="${-(90-8.277)*M_PI/180} 0 ${-90*M_PI/180}" />
+    <origin xyz="0 0 0" rpy="${-90*M_PI/180} 0 ${-90*M_PI/180}" />
   </joint>
   <link name="$(arg prefix)/camera_optical_frame">
